Commit message: Real Part 2 Final

File: install/prac1_robot_description/share/prac1_robot_description/src/description/robot.urdf (robot description, URDF)
Before this commit: robot diff_drive_robot, 6 links, 5 joints
Joints:
- joint left_wheel_joint: origin xyz=0 0.25 0.1 -> xyz=0 0.25 0.1 rpy=0 0 0; parent base_link -> base_footprint
- joint right_wheel_joint: origin xyz=0 -0.25 0.1 -> xyz=0 -0.25 0.1 rpy=0 0 0; parent base_link -> base_footprint

File: prac1_robot_description/src/description/robot.urdf (robot description, URDF)
Before this commit: robot diff_drive_robot, 6 links, 5 joints
Joints:
- joint left_wheel_joint: origin xyz=0 0.25 0.1 -> xyz=0 0.25 0.1 rpy=0 0 0; parent base_link -> base_footprint
- joint right_wheel_joint: origin xyz=0 -0.25 0.1 -> xyz=0 -0.25 0.1 rpy=0 0 0; parent base_link -> base_footprint
